File: ESP32/ESP32.kicad_pcb (KiCad board)
At the start: 2 copper layers, 4 parts

Commit message: Add files via upload
Connected secondary RX and TX
Routing:
- net (no net): track 74.5 -> 171.4 mm
- added copper zone on B.Cu, net (none)
Other:
- board outline added: 68.6 x 27.9 mm
Changed lines of the file:
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@@
     (pad_to_mask_clearance 0)
     (pcbplotparams
-      (layerselection 0x0001000_ffffffff)
+      (layerselection 0x00010c0_ffffffff)
       (plot_on_all_layers_selection 0x0000000_00000000)
       (disableapertmacros false)
@@
     )
   )
-  (segment (start 162.55 106.69) (end 160.01 109.23) (width 0) (layer "B.Cu") (net 0))
-  (segment (start 175.25 104.15) (end 170.17 109.23) (width 0) (layer "B.Cu") (net 0))
-  (segment (start 162.55 109.23) (end 162.55 111.77) (width 0) (layer "B.Cu") (net 0))
-  (segment (start 175.25 101.61) (end 175.25 104.15) (width 0) (layer "B.Cu") (net 0))
-  (segment (start 170.18 91.44) (end 165.09 96.53) (width 0) (layer "B.Cu") (net 0))
-  (segment (start 165.09 96.53) (end 154.93 96.53) (width 0) (layer "B.Cu") (net 0))
-  (segment (start 160.01 109.23) (end 160.01 111.77) (width 0) (layer "B.Cu") (net 0))
-  (segment (start 152.39 99.07) (end 152.39 101.61) (width 0) (layer "B.Cu") (net 0))
-  (segment (start 162.55 101.61) (end 162.55 106.69) (width 0) (layer "B.Cu") (net 0))
-  (segment (start 137.16 93.98) (end 134.61 96.53) (width 0) (layer "B.Cu") (net 0))
-  (segment (start 165.09 101.61) (end 165.09 106.69) (width 0) (layer "B.Cu") (net 0))
-  (segment (start 165.09 106.69) (end 162.55 109.23) (width 0) (layer "B.Cu") (net 0))
-  (segment (start 154.93 96.53) (end 152.39 99.07) (width 0) (layer "B.Cu") (net 0))
-  (segment (start 170.17 109.23) (end 170.17 111.77) (width 0) (layer "B.Cu") (net 0))
-  (segment (start 137.16 88.885) (end 137.16 93.98) (width 0) (layer "B.Cu") (net 0))
-  (segment (start 170.18 88.885) (end 170.18 91.44) (width 0) (layer "B.Cu") (net 0))
-  (segment (start 134.61 96.53) (end 134.61 101.585) (width 0) (layer "B.Cu") (net 0))
-  (zone (net 0) (net_name "") (layer "F.Cu") (hatch edge 0.5)
-    (priority 1)
+  (gr_line (start 180.34 114.3) (end 180.34 86.36)
+    (stroke (width 0.1) (type default)) (layer "Edge.Cuts"))
+  (gr_line (start 111.76 114.3) (end 180.34 114.3)
+    (stroke (width 0.1) (type default)) (layer "Edge.Cuts"))
+  (gr_line (start 180.34 86.36) (end 111.76 86.36)
+    (stroke (width 0.1) (type default)) (layer "Edge.Cuts"))
+  (gr_line (start 111.76 86.36) (end 111.76 114.3)
+    (stroke (width 0.1) (type default)) (layer "Edge.Cuts"))
+  (segment (start 149.86 96.52) (end 165.1 96.52) (width 0.5) (layer "F.Cu") (net 0))
+  (segment (start 165.1 96.52) (end 167.64 99.06) (width 0.5) (layer "F.Cu") (net 0))
+  (segment (start 132.08 88.885) (end 132.08 91.44) (width 0.5) (layer "F.Cu") (net 0))
+  (segment (start 134.62 93.98) (end 147.32 93.98) (width 0.5) (layer "F.Cu") (net 0))
+  (segment (start 167.63 99.07) (end 167.63 101.61) (width 0.5) (layer "F.Cu") (net 0))
+  (segment (start 170.17 101.61) (end 170.17 104.13) (width 0.5) (layer "F.Cu") (net 0))
+  (segment (start 132.08 91.44) (end 134.62 93.98) (width 0.5) (layer "F.Cu") (net 0))
+  (segment (start 170.18 104.14) (end 167.64 106.68) (width 0.5) (layer "F.Cu") (net 0))
+  (segment (start 167.64 99.06) (end 167.63 99.07) (width 0.5) (layer "F.Cu") (net 0))
+  (segment (start 147.32 93.98) (end 149.86 96.52) (width 0.5) (layer "F.Cu") (net 0))
+  (segment (start 129.54 91.44) (end 129.54 88.885) (width 0.5) (layer "F.Cu") (net 0))
+  (segment (start 144.78 106.68) (end 129.54 91.44) (width 0.5) (layer "F.Cu") (net 0))
+  (segment (start 170.17 104.13) (end 170.18 104.14) (width 0.5) (layer "F.Cu") (net 0))
+  (segment (start 167.64 106.68) (end 144.78 106.68) (width 0.5) (layer "F.Cu") (net 0))
+  (segment (start 162.55 109.23) (end 162.55 111.77) (width 0.5) (layer "B.Cu") (net 0))
+  (segment (start 152.39 99.07) (end 152.39 101.61) (width 0.5) (layer "B.Cu") (net 0))
+  (segment (start 170.18 88.885) (end 170.18 91.44) (width 0.5) (layer "B.Cu") (net 0))
+  (segment (start 165.09 101.61) (end 165.09 106.67) (width 0.5) (layer "B.Cu") (net 0))
+  (segment (start 162.56 106.68) (end 160.01 109.23) (width 0.5) (layer "B.Cu") (net 0))
+  (segment (start 157.48 93.98) (end 152.39 99.07) (width 0.5) (layer "B.Cu") (net 0))
+  (segment (start 165.09 106.67) (end 165.1 106.68) (width 0.5) (layer "B.Cu") (net 0))
+  (segment (start 175.26 104.14) (end 170.17 109.23) (width 0.5) (layer "B.Cu") (net 0))
+  (segment (start 167.64 93.98) (end 157.48 93.98) (width 0.5) (layer "B.Cu") (net 0))
+  (segment (start 175.25 104.13) (end 175.26 104.14) (width 0.5) (layer "B.Cu") (net 0))
+  (segment (start 162.55 106.67) (end 162.56 106.68) (width 0.5) (layer "B.Cu") (net 0))
+  (segment (start 134.61 96.53) (end 134.61 101.585) (width 0.5) (layer "B.Cu") (net 0))
+  (segment (start 170.18 91.44) (end 167.64 93.98) (width 0.5) (layer "B.Cu") (net 0))
+  (segment (start 165.1 106.68) (end 162.55 109.23) (width 0.5) (layer "B.Cu") (net 0))
+  (segment (start 170.17 109.23) (end 170.17 111.77) (width 0.5) (layer "B.Cu") (net 0))
+  (segment (start 137.16 88.885) (end 137.16 93.98) (width 0.5) (layer "B.Cu") (net 0))
+  (segment (start 137.16 93.98) (end 134.61 96.53) (width 0.5) (layer "B.Cu") (net 0))
+  (segment (start 162.55 101.61) (end 162.55 106.67) (width 0.5) (layer "B.Cu") (net 0))
+  (segment (start 175.25 101.61) (end 175.25 104.13) (width 0.5) (layer "B.Cu") (net 0))
+  (segment (start 160.01 109.23) (end 160.01 111.77) (width 0.5) (layer "B.Cu") (net 0))
+  (zone (net 0) (net_name "") (layers "F&B.Cu") (hatch edge 0.5)
     (connect_pads (clearance 0.5))
     (min_thickness 0.25) (filled_areas_thickness no)
@@
     (polygon
       (pts
-        (xy 111.75 83.83)
-        (xy 111.75 116.85)
-        (xy 180.33 116.85)
-        (xy 180.33 83.83)
+        (xy 111.76 86.36)
+        (xy 111.76 114.3)
+        (xy 180.34 114.3)
+        (xy 180.34 86.36)
       )
     )

Commit message: Add files via upload
Made proper Rx Tx connection
Routing:
- net (no net): track 171.4 -> 139.7 mm
Changed lines of the file:
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@@
   (gr_line (start 111.76 86.36) (end 111.76 114.3)
     (stroke (width 0.1) (type default)) (layer "Edge.Cuts"))
-  (segment (start 149.86 96.52) (end 165.1 96.52) (width 0.5) (layer "F.Cu") (net 0))
-  (segment (start 165.1 96.52) (end 167.64 99.06) (width 0.5) (layer "F.Cu") (net 0))
-  (segment (start 132.08 88.885) (end 132.08 91.44) (width 0.5) (layer "F.Cu") (net 0))
-  (segment (start 134.62 93.98) (end 147.32 93.98) (width 0.5) (layer "F.Cu") (net 0))
-  (segment (start 167.63 99.07) (end 167.63 101.61) (width 0.5) (layer "F.Cu") (net 0))
-  (segment (start 170.17 101.61) (end 170.17 104.13) (width 0.5) (layer "F.Cu") (net 0))
-  (segment (start 132.08 91.44) (end 134.62 93.98) (width 0.5) (layer "F.Cu") (net 0))
-  (segment (start 170.18 104.14) (end 167.64 106.68) (width 0.5) (layer "F.Cu") (net 0))
-  (segment (start 167.64 99.06) (end 167.63 99.07) (width 0.5) (layer "F.Cu") (net 0))
-  (segment (start 147.32 93.98) (end 149.86 96.52) (width 0.5) (layer "F.Cu") (net 0))
-  (segment (start 129.54 91.44) (end 129.54 88.885) (width 0.5) (layer "F.Cu") (net 0))
-  (segment (start 144.78 106.68) (end 129.54 91.44) (width 0.5) (layer "F.Cu") (net 0))
-  (segment (start 170.17 104.13) (end 170.18 104.14) (width 0.5) (layer "F.Cu") (net 0))
-  (segment (start 167.64 106.68) (end 144.78 106.68) (width 0.5) (layer "F.Cu") (net 0))
+  (segment (start 142.23 111.77) (end 142.23 109.23) (width 0.5) (layer "F.Cu") (net 0))
+  (segment (start 170.18 104.14) (end 170.17 104.13) (width 0.5) (layer "F.Cu") (net 0))
+  (segment (start 144.77 109.295359) (end 145.421548 108.643811) (width 0.5) (layer "F.Cu") (net 0))
+  (segment (start 144.78 106.68) (end 165.1 106.68) (width 0.5) (layer "F.Cu") (net 0))
+  (segment (start 167.63 104.15) (end 167.63 101.61) (width 0.5) (layer "F.Cu") (net 0))
+  (segment (start 165.1 106.68) (end 167.63 104.15) (width 0.5) (layer "F.Cu") (net 0))
+  (segment (start 145.421548 108.643811) (end 165.676189 108.643811) (width 0.5) (layer "F.Cu") (net 0))
+  (segment (start 165.676189 108.643811) (end 170.18 104.14) (width 0.5) (layer "F.Cu") (net 0))
+  (segment (start 142.23 109.23) (end 144.78 106.68) (width 0.5) (layer "F.Cu") (net 0))
+  (segment (start 170.17 104.13) (end 170.17 101.61) (width 0.5) (layer "F.Cu") (net 0))
+  (segment (start 144.77 111.77) (end 144.77 109.295359) (width 0.5) (layer "F.Cu") (net 0))
   (segment (start 162.55 109.23) (end 162.55 111.77) (width 0.5) (layer "B.Cu") (net 0))
   (segment (start 152.39 99.07) (end 152.39 101.61) (width 0.5) (layer "B.Cu") (net 0))
